Commit message: aaa

File: car/urdf/car.xacro (robot description, xacro)
@@ -1,14 +1,15 @@
 <?xml version="1.0"?>
-<robot name="fourwheelrobot" xmlns:xacro="http://www.ros.org/wiki/xacro" >
+<robot name="car" xmlns:xacro="http://www.ros.org/wiki/xacro" >
     <xacro:property name="radius" value="0.2" />
     <xacro:property name="wheel" value="wheel" />
+    <xacro:include filename="$(find car)/urdf/car.gazebo" />
     <xacro:macro name="wheel_macro" params="rpy name joint_origin_xyz">
         <link name="${name}">
           <inertial>
-            <origin xyz="0 0 0.5" rpy="${rpy}" />
+            <origin xyz="0 0 0.0" rpy="${rpy}" />
             <mass value="1.0"/>
-            <inertia ixx="0.0" ixy="0.0" ixz="0.0" iyy="0.0" iyz="0.0" izz="0.0"/>
+            <inertia ixx="1.0" ixy="1.0" ixz="1.0" iyy="1.0" iyz="1.0" izz="1.0"/>
           </inertial>
-          <visual name="">
+          <visual>
               <origin xyz="0 0 0" rpy="${rpy}" />
               <geometry>
@@ -27,27 +28,29 @@
           </collision>
         </link>
-        <joint name="joint_${name}" type="continuous">
+        <joint name="joint_${name}" type="continuous">  <!--continuous--> <!--revolute-->
           <parent link="base_link"/>
           <child link="${name}"/>
           <origin xyz="${joint_origin_xyz}" rpy="0 0 0" />
           <axis xyz="0 1 0" rpy="0 0 0" />
+          <limit upper="6.28" lower="-6.28" effort="1000" velocity="1000.00"/>
         </joint>
-        <gazebo reference="${name}">
-          <mu1 value="200.0"/>
-          <mu2 value="100.0"/>
-          <kp value="10000000.0" />
-          <kd value="1.0" />
-          <material>Gazebo/Grey</material>
-        </gazebo>
         <transmission name="trnasm_${name}">
           <type>transmission_interface/SimpleTransmission</type>
-          <actuator name="$act_${name}">
+          <actuator name="act_${name}">
             <mechanicalReduction>1</mechanicalReduction>
           </actuator>
           <joint name="joint_${name}">
-            <hardwareInterface>VelocityJointInterface</hardwareInterface>
+            <hardwareInterface>EffortJointInterface</hardwareInterface>
+            <!--hardwareInterface>VelocityJointInterface</hardwareInterface-->
+            <!--hardwareInterface>hardware_interface/PositionJointInterface</hardwareInterface-->
           </joint>
         </transmission>
     </xacro:macro>
+  <!-- Used for fixing robot to Gazebo 'base_link' -->
+  <link name="world"/>
+  <joint name="fixed" type="fixed">
+    <parent link="world"/>
+    <child link="base_link"/>
+  </joint>
   <!-- Base link -->
   <link name="base_link">
@@ -70,16 +73,3 @@
   <!-- Back Left Wheel -->
   <xacro:wheel_macro rpy="1.570795 0 0" name="b_l_${wheel}" joint_origin_xyz="-0.25 0.30 0" />
-  <!-- Gazebo plugin for ROS Control -->
-  <gazebo>
-    <plugin name="gazebo_ros_control" filename="libgazebo_ros_control.so">
-        <robotNamespace>/mugator_manip</robotNamespace>
-        <robotSimType>gazebo_ros_control/DefaultRobotHWSim</robotSimType>
-        <legacyModeNS>true</legacyModeNS>
-    </plugin>
-  </gazebo>
-  </robot>
-    <!-- <gazebo>
-    <plugin name="gazebo_ros_control" filename="libgazebo_ros_control.so">
-      <robotNamespace>/</robotNamespace>
-    </plugin>
-  </gazebo> -->
+</robot>

Commit message: !

File: car/urdf/car.xacro (robot description, xacro)
@@ -1,3 +1,4 @@
 <?xml version="1.0"?>
+<!-- http://wiki.ros.org/ros_control#Controllers -->
 <robot name="car" xmlns:xacro="http://www.ros.org/wiki/xacro" >
     <xacro:property name="radius" value="0.2" />
@@ -33,5 +34,5 @@
           <origin xyz="${joint_origin_xyz}" rpy="0 0 0" />
           <axis xyz="0 1 0" rpy="0 0 0" />
-          <limit upper="6.28" lower="-6.28" effort="1000" velocity="1000.00"/>
+          <!--limit upper="6.28" lower="-6.28" effort="1000" velocity="1000.00"/-->
         </joint>
         <transmission name="trnasm_${name}">
@@ -39,7 +40,8 @@
           <actuator name="act_${name}">
             <mechanicalReduction>1</mechanicalReduction>
+            <hardwareInterface>hhardware_interface/EffortJointInterface</hardwareInterface>
           </actuator>
           <joint name="joint_${name}">
-            <hardwareInterface>EffortJointInterface</hardwareInterface>
+            <hardwareInterface>hardware_interface/EffortJointInterface</hardwareInterface>
             <!--hardwareInterface>VelocityJointInterface</hardwareInterface-->
             <!--hardwareInterface>hardware_interface/PositionJointInterface</hardwareInterface-->

Commit message: 1

File: car/urdf/car.xacro (robot description, xacro)
@@ -1,77 +1,241 @@
 <?xml version="1.0"?>
-<!-- http://wiki.ros.org/ros_control#Controllers -->
-<robot name="car" xmlns:xacro="http://www.ros.org/wiki/xacro" >
-    <xacro:property name="radius" value="0.2" />
-    <xacro:property name="wheel" value="wheel" />
+<robot
+    xmlns:gazebo="http://playerstage.sourceforge.net/gazebo/xmlschema/#gz"
+    xmlns:model="http://playerstage.sourceforge.net/gazebo/xmlschema/#model"
+    xmlns:sensor="http://playerstage.sourceforge.net/gazebo/xmlschema/#sensor"
+    xmlns:body="http://playerstage.sourceforge.net/gazebo/xmlschema/#body"
+    xmlns:geom="http://playerstage.sourceforge.net/gazebo/xmlschema/#geom"
+    xmlns:joint="http://playerstage.sourceforge.net/gazebo/xmlschema/#joint"
+    xmlns:controller="http://playerstage.sourceforge.net/gazebo/xmlschema/#controller"
+    xmlns:interface="http://playerstage.sourceforge.net/gazebo/xmlschema/#interface"
+    xmlns:rendering="http://playerstage.sourceforge.net/gazebo/xmlschema/#rendering"
+    xmlns:physics="http://playerstage.sourceforge.net/gazebo/xmlschema/#physics"
+    xmlns:xacro="http://www.ros.org/wiki/xacro"
+    name="car">
     <xacro:include filename="$(find car)/urdf/car.gazebo" />
-    <xacro:macro name="wheel_macro" params="rpy name joint_origin_xyz">
-        <link name="${name}">
-          <inertial>
-            <origin xyz="0 0 0.0" rpy="${rpy}" />
-            <mass value="1.0"/>
-            <inertia ixx="1.0" ixy="1.0" ixz="1.0" iyy="1.0" iyz="1.0" izz="1.0"/>
-          </inertial>
-          <visual>
-              <origin xyz="0 0 0" rpy="${rpy}" />
-              <geometry>
-                <cylinder length="0.1" radius="${radius}" />
-              </geometry>
-              <material name="black">
-                <color rgba="0.05 0.05 0.05 1"/>
-              <texture filename=""/>
-            </material>
-          </visual>
-          <collision>
-            <origin xyz="0 0 0" rpy="${rpy}" />
-            <geometry>
-              <cylinder length="0.1" radius="${radius}" />
-            </geometry>
-          </collision>
-        </link>
-        <joint name="joint_${name}" type="continuous">  <!--continuous--> <!--revolute-->
-          <parent link="base_link"/>
-          <child link="${name}"/>
-          <origin xyz="${joint_origin_xyz}" rpy="0 0 0" />
-          <axis xyz="0 1 0" rpy="0 0 0" />
-          <!--limit upper="6.28" lower="-6.28" effort="1000" velocity="1000.00"/-->
-        </joint>
-        <transmission name="trnasm_${name}">
-          <type>transmission_interface/SimpleTransmission</type>
-          <actuator name="act_${name}">
-            <mechanicalReduction>1</mechanicalReduction>
-            <hardwareInterface>hhardware_interface/EffortJointInterface</hardwareInterface>
-          </actuator>
-          <joint name="joint_${name}">
-            <hardwareInterface>hardware_interface/EffortJointInterface</hardwareInterface>
-            <!--hardwareInterface>VelocityJointInterface</hardwareInterface-->
-            <!--hardwareInterface>hardware_interface/PositionJointInterface</hardwareInterface-->
-          </joint>
-        </transmission>
-    </xacro:macro>
-  <!-- Used for fixing robot to Gazebo 'base_link' -->
-  <link name="world"/>
-  <joint name="fixed" type="fixed">
-    <parent link="world"/>
-    <child link="base_link"/>
-  </joint>
-  <!-- Base link -->
-  <link name="base_link">
-    <visual>
-      <origin xyz="0 0 0.1" rpy="0 0 0" />
-      <geometry>
-          <box size="1 0.5 0.35"/>
-      </geometry>
-      <material name="yellow">
-        <color rgba="0.8 0.8 0 1"/>
-      </material>
-    </visual>
-  </link>
-  <!-- Front Right Wheel -->
-  <xacro:wheel_macro rpy="1.570795 0 0" name="f_r_${wheel}" joint_origin_xyz="0.25 -0.30 0"/>
-  <!-- Back Right Wheel -->
-  <xacro:wheel_macro rpy="1.570795 0 0" name="b_r_${wheel}" joint_origin_xyz="-0.25 -0.30 0"/>
-  <!-- Front Left Wheel -->
-  <xacro:wheel_macro rpy="1.570795 0 0" name="f_l_${wheel}" joint_origin_xyz="0.25 0.30 0"/>
-  <!-- Back Left Wheel -->
-  <xacro:wheel_macro rpy="1.570795 0 0" name="b_l_${wheel}" joint_origin_xyz="-0.25 0.30 0" />
+    <xacro:property name="M_PI" value="3.1415926535897931" />
+    <xacro:property name="carLength" value="0.3" />
+    <xacro:property name="carWidth" value="0.15" />
+    <xacro:property name="carHeight" value="0.1" />
+    <xacro:property name="wheelRadius" value="0.06" />
+    <xacro:property name="wheelWidth" value="0.025" />
+    <!-- Main body -->
+    <link name="base_link">
+        <inertial>
+            <mass value="0.2" />
+            <origin xyz="0 0 0" />
+            <inertia  ixx="0.2" ixy="0.0"  ixz="0.0"  iyy="0.2"  iyz="0.0"  izz="0.2" />
+        </inertial>
+        <visual>
+            <origin xyz="0 0 0" rpy="0 0 0" />
+            <geometry>
+                <box size="${carLength} ${carWidth} ${carHeight}" />
+            </geometry>
+            <material name="Red"/>
+        </visual>
+        <collision>
+            <origin xyz="0 0 0" rpy="0 0 0" />
+            <geometry>
+                <box size="${carLength} ${carWidth} ${carHeight}" />
+            </geometry>
+        </collision>
+    </link>
+	<!-- the front left wheel -->
+    <joint name="front_left_wheel_joint" type="revolute" >
+        <axis xyz="0 0 1" />
+        <parent link="base_link" />
+        <child link="front_left_wheel_link" />
+        <origin xyz="0.16 0.1 -0.1" rpy="0 0 0" />
+        <limit effort="1000.0" lower="-0.5" upper="0.5" velocity="0.5"/>
+    </joint>
+    <link name="front_left_wheel_link">
+        <inertial>
+            <mass value="0.01" />
+            <origin xyz="0 0 0" />
+            <inertia  ixx="0.01" ixy="0.0"  ixz="0.0"  iyy="0.01"  iyz="0.0"  izz="0.01" />
+        </inertial>
+        <visual>
+            <origin xyz="0 0 0" rpy="${M_PI/2} 0 0" />
+            <geometry>
+                <cylinder radius="${wheelRadius}" length="${wheelWidth}" />
+            </geometry>
+            <material name="Green"/>
+        </visual>
+        <collision>
+            <origin xyz="0 0 0" rpy="${M_PI/2} 0 0" />
+            <geometry>
+                <cylinder radius="${wheelRadius}" length="${wheelWidth}" />
+            </geometry>
+        </collision>
+    </link>
+    <transmission name="trnasm_front_left_wheel_joint">
+      <type>transmission_interface/SimpleTransmission</type>
+      <actuator name="act_front_left_wheel_joint">
+        <mechanicalReduction>1</mechanicalReduction>
+        <hardwareInterface>hardware_interface/VelocityJointInterface</hardwareInterface>
+      </actuator>
+      <joint name="front_left_wheel_joint">
+        <hardwareInterface>hardware_interface/VelocityJointInterface</hardwareInterface>
+      </joint>
+    </transmission>
+	<!-- the front right wheel -->
+    <joint name="front_right_wheel_joint" type="revolute" >
+        <axis xyz="0 0 1" />
+        <parent link="base_link" />
+        <child link="front_right_wheel_link" />
+        <origin xyz="0.16 -0.1 -0.1" rpy="0 0 0" />
+        <limit effort="1000.0" lower="-0.5" upper="0.5" velocity="0.5"/>
+    </joint>
+    <link name="front_right_wheel_link">
+        <inertial>
+            <mass value="0.01" />
+            <origin xyz="0 0 0" />
+            <inertia  ixx="0.01" ixy="0.0"  ixz="0.0"  iyy="0.01"  iyz="0.0"  izz="0.01" />
+        </inertial>
+        <visual>
+            <origin xyz="0 0 0" rpy="${M_PI/2} 0 0" />
+            <geometry>
+                <cylinder radius="${wheelRadius}" length="${wheelWidth}" />
+            </geometry>
+            <material name="Green"/>
+        </visual>
+        <collision>
+            <origin xyz="0 0 0" rpy="${M_PI/2} 0 0" />
+            <geometry>
+                <cylinder radius="${wheelRadius}" length="${wheelWidth}" />
+            </geometry>
+        </collision>
+    </link>
+    <transmission name="trnasm_front_right_wheel">
+      <type>transmission_interface/SimpleTransmission</type>
+      <actuator name="act_front_right_wheel">
+        <mechanicalReduction>1</mechanicalReduction>
+        <hardwareInterface>hardware_interface/VelocityJointInterface</hardwareInterface>
+      </actuator>
+      <joint name="front_right_wheel_joint">
+        <hardwareInterface>hardware_interface/VelocityJointInterface</hardwareInterface>
+      </joint>
+    </transmission>
+	<!-- the back left wheel -->
+    <joint name="back_left_wheel_joint" type="continuous" >
+        <axis xyz="0 1 0" />
+        <parent link="base_link" />
+        <child link="back_left_wheel_link" />
+        <origin xyz="-0.16 0.1 -0.1" rpy="0 0 0" />
+    </joint>
+    <link name="back_left_wheel_link">
+        <inertial>
+            <mass value="0.01" />
+            <origin xyz="0 0 0" />
+            <inertia  ixx="0.01" ixy="0.0"  ixz="0.0"  iyy="0.01"  iyz="0.0"  izz="0.01" />
+        </inertial>
+        <visual>
+            <origin xyz="0 0 0" rpy="${M_PI/2} 0 0" />
+            <geometry>
+                <cylinder radius="${wheelRadius}" length="${wheelWidth}" />
+            </geometry>
+            <material name="Black"/>
+        </visual>
+        <collision>
+            <origin xyz="0 0 0" rpy="${M_PI/2} 0 0" />
+            <geometry>
+                <cylinder radius="${wheelRadius}" length="${wheelWidth}" />
+            </geometry>
+        </collision>
+    </link>
+    <transmission name="trnasm_back_left_wheel">
+      <type>transmission_interface/SimpleTransmission</type>
+      <actuator name="act_back_left_wheel">
+        <mechanicalReduction>1</mechanicalReduction>
+        <hardwareInterface>hardware_interface/VelocityJointInterface</hardwareInterface>
+      </actuator>
+      <joint name="back_left_wheel_joint">
+        <hardwareInterface>hardware_interface/VelocityJointInterface</hardwareInterface>
+      </joint>
+    </transmission>
+	<!-- the back right wheel -->
+    <joint name="back_right_wheel_joint" type="continuous" >
+        <axis xyz="0 1 0" />
+        <parent link="base_link" />
+        <child link="back_right_wheel_link" />
+        <origin xyz="-0.16 -0.1 -0.1" rpy="0 0 0" />
+    </joint>
+    <link name="back_right_wheel_link">
+        <inertial>
+            <mass value="0.01" />
+            <origin xyz="0 0 0" />
+            <inertia  ixx="0.01" ixy="0.0"  ixz="0.0"  iyy="0.01"  iyz="0.0"  izz="0.01" />
+        </inertial>
+        <visual>
+            <origin xyz="0 0 0" rpy="${M_PI/2} 0 0" />
+            <geometry>
+                <cylinder radius="${wheelRadius}" length="${wheelWidth}" />
+            </geometry>
+            <material name="Black"/>
+        </visual>
+        <collision>
+            <origin xyz="0 0 0" rpy="${M_PI/2} 0 0" />
+            <geometry>
+                <cylinder radius="${wheelRadius}" length="${wheelWidth}" />
+            </geometry>
+        </collision>
+    </link>
+    <transmission name="trnasm_back_right_wheel">
+      <type>transmission_interface/SimpleTransmission</type>
+      <actuator name="act_back_right_wheel">
+        <mechanicalReduction>1</mechanicalReduction>
+        <hardwareInterface>hardware_interface/VelocityJointInterface</hardwareInterface>
+      </actuator>
+      <joint name="back_right_wheel_joint">
+        <hardwareInterface>hardware_interface/VelocityJointInterface</hardwareInterface>
+      </joint>
+    </transmission>
+    <joint name="laser_base_mount_joint" type="fixed">
+        <origin xyz="0 0 0.05" rpy="0 0 0" />
+        <parent link="base_link"/>
+        <child link="laser_base_link"/>
+    </joint>
+    <link name="laser_base_link" type="fixed">
+        <inertial>
+            <mass value="0.1"/>
+            <origin xyz="0 0 0.0"/>
+            <inertia ixx="0.1" ixy="0" ixz="0" iyy="0.1" iyz="0" izz="0.1"/>
+        </inertial>
+        <visual>
+            <origin rpy="0 0 0" xyz="0 0 0.025"/>
+            <geometry>
+                <box size="0.05 0.05 0.05"/>
+            </geometry>
+        </visual>
+        <collision>
+            <origin rpy="0 0 0" xyz="0 0 0.025"/>
+            <geometry>
+                <box size="0.05 0.05 0.05"/>
+            </geometry>
+        </collision>
+    </link>
+    <joint name="base_scan_joint" type="fixed" >
+        <origin xyz="0 0 0.05" rpy="0 0 0" />
+        <parent link="laser_base_link" />
+        <child link="base_scan_link"/>
+    </joint>
+    <link name="base_scan_link" type="laser">
+        <inertial>
+            <mass value="0.1"/>
+            <origin xyz="0 0 0.0"/>
+            <inertia ixx="0.1" ixy="0" ixz="0" iyy="0.1" iyz="0" izz="0.1"/>
+        </inertial>
+        <visual>
+            <origin rpy="0 0 0" xyz="0 0 0.014"/>
+            <geometry>
+                <cylinder radius="0.0229" length="0.028"/>
+            </geometry>
+        </visual>
+        <collision>
+            <origin rpy="0 0 0" xyz="0 0 0.014"/>
+            <geometry>
+                <cylinder radius="0.0229" length="0.028"/>
+            </geometry>
+        </collision>
+    </link>
 </robot>
